File: PC104-ISA-Card.kicad_sch (KiCad schematic)
At the start: 4 parts, among them J1 Bus_PC104_16bit, J2 Bus_ISA_16bit

Commit message: Preliminary schematic
Parts:
- added B1: Bracket, symbol local:Bracket
- added C1, C3, C5, C7: 10u, Capacitor_Tantalum_SMD:CP_EIA-7343-15_Kemet-W, symbol Device:C_Polarized_Small
- added C2, C4, C6, C8: 100n, Capacitor_SMD:C_0603_1608Metric, symbol Device:C_Small
Connections:
- net +12V: now also C3.1, C4.1
- net +5V: now also C1.1, C2.1
- net -12V: now also C5.2, C6.2
- net -5V: now also C7.2, C8.2
- net BA1/SA1: now also J1.A30 (SA1); no longer J1.A20 (SA11)
- net GND: now also C1.2, C2.2, C3.2, C4.2, C5.1, C6.1, C7.1, C8.1
- net ~{SRDY}: now also J2.8 (UNUSED)
- no-connect marks 1 -> 0
Other:
- title: (none) -> PC/104 ISA Card
- moved on the sheet: H1, H2, J1, J2
